File: HARDWARE/NP001 - Placa Host/MB_V2.sch (KiCad schematic (older format))
At the start: 38 parts, among them J10 GPS/GPRS, J11 TP_RX_PIC, J12 TP_SDO, J13 TP_SCK, J14 DM3CS-SF, J15 Sensor_SO2, J16 Sensor_O3, J17 Sensor_NO2, J18 Sensor_PM10, J2 Datos_LORA, J3 Salida_Bomba, J4 Sensor_CO, J5 POWER_MB, J6 TP_SCL, J7 PICKIT3, J8 TP_SDA, J9 TP_TX_PIC, Q1 BC807, U1 AP1117-33, U3 PIC24FJ64GB002-I/P, Y1 8MHz

Commit message: Daniel Prieto:
-Subo placa enviada a China.
Parts:
- removed J5: POWER_MB, Connectors_JST:JST_PH_B2B-PH-SM4-TB_02x2.00mm_Straight, symbol Conn_01x02
- added C1, C3: 0.1u, Capacitors_SMD:C_0805, symbol C
- added C2: 10u, Capacitors_SMD:C_0805, symbol C
- added C4, C5: 28u, Capacitors_SMD:C_1206, symbol C
- added D1: LED_RCGB, LEDs:LED_D5.0mm-4, symbol LED_RAGB
- added D5: SS34, Diodes_SMD:D_SMC, symbol D_Zener
- added J10: BAT-, Mounting_Holes:MountingHole_2.2mm_M2_DIN965_Pad, symbol Conn_01x01
- added J3: Entrada_Alimentacion, Connectors_USB:USB_Micro-B_Molex_47346-0001, symbol Conn_01x05
- added J9: BAT+, Mounting_Holes:MountingHole_2.2mm_M2_DIN965_Pad, symbol Conn_01x01
- added L1: 22u, Inductors_SMD:L_10.4x10.4_H4.8, symbol L
- added R1: 1.2k, Resistors_SMD:R_0805, symbol R
- added R12: 18k, Resistors_SMD:R_0805, symbol R
- added R13, R20: 2.2k, Resistors_SMD:R_0805, symbol R
- added R14: 180k, Resistors_SMD:R_0805, symbol R
- added R19: 3.3k, Resistors_SMD:R_0805, symbol R
- added R2, R3, R4: 1k, Resistors_SMD:R_0805, symbol R
- added R6: 100, Resistors_SMD:R_0805, symbol R
- added U1: TP4056, Housings_SOIC:SOIC-8_3.9x4.9mm_Pitch1.27mm, symbol TP4056
- added U2: DW01-P, Housings_SSOP:TSOP-6_1.65x3.05mm_Pitch0.95mm, symbol DW01-P
- added U3: 8205A, Housings_SSOP:TSSOP-8_4.4x3mm_Pitch0.65mm, symbol 8205A
- added U5: MT3608, Housings_SSOP:TSOP-6_1.65x3.05mm_Pitch0.95mm, symbol MT3608
- D3: renamed from D1; footprint LEDs:LED_0805_HandSoldering -> LEDs:LED_D3.0mm_Horizontal_O1.27mm_Z2.0mm
- D4: renamed from D2; footprint LEDs:LED_0805_HandSoldering -> LEDs:LED_D3.0mm_Horizontal_O1.27mm_Z2.0mm
- renumbered C5 to C10, C9 to C6, C10 to C7, C11 to C8, C1 to C9, J2 to J1, J6 to J11, J7 to J12, J8 to J13, J9 to J15, J10 to J16, J11 to J17, J12 to J18, J13 to J19, J3 to J2, J14 to J20, J15 to J5, J16 to J6, J17 to J7, J18 to J8, R9 to R10, R10 to R11, R11 to R15, R12 to R16, R13 to R17, R14 to R18, R4 to R5, R6 to R7, R7 to R8, R8 to R9, U3 to U4, U1 to U6
Connections:
- net +5V: now also C1.1, D1.2 (A), J3.1 (Pin_1), U1.4 (VCC), U1.8 (CE); no longer J16.1 (Pin_1), J4.3 (Pin_3), J5.3 (Pin_3), J6.3 (Pin_3), J7.3 (Pin_3), J8.3 (Pin_3), Q1.2 (E), U6.3 (VI)
- net GND: now also C1.2, C2.2, C4.2, C5.2, J3.5 (Pin_5), R1.1, R13.2, R20.2, R4.2, U1.1 (TEMP), U1.3 (GND), U3.2 (S1), U3.3 (S1), U5.2 (GND)
- net V_BAT: now reaches U4.12 (C2INC/RA4)
- net V_BAT: now also R19.2, R20.1
- new net: R1.2, U1.2 (PROG)
- new net: R3.2, U1.6 (nSTDBY)
- new net: R2.2, U1.7 (nCHRG)
- new net: D1.4 (BK), R3.1
- new net: D1.1 (RK), R2.1
- new net: R4.1, U2.2 (CS)
- new net: C3.1, R6.2, U2.5 (VCC)
- new net: U2.1 (OD), U3.5 (G2)
- new net: U2.3 (OC), U3.4 (G1)
- new net: C3.2, J10.1 (Pin_1), U2.6 (GND), U3.6 (S2), U3.7 (S2)
- new net: D5.2 (A), L1.1, U5.1 (SW)
- new net: R12.2, R13.1, R14.2, U5.3 (FB)
- new net BAT+: C2.1, C5.1, J9.1 (Pin_1), L1.2, R19.1, R6.1, U1.5 (BAT), U5.4 (EN), U5.5 (IN)
- new net VDD2: C4.1, D5.1 (K), J16.1 (Pin_1), J4.3 (Pin_3), J5.3 (Pin_3), J6.3 (Pin_3), J7.3 (Pin_3), J8.3 (Pin_3), Q1.2 (E), R12.1, R14.1, U6.3 (VI)
- no-connect marks 31 -> 38
Other:
- note added: "Cargador\n"
- note added: "ELEVADOR 1"
- note added: "I_max ="
- note added: "Ibat = Vprog x 1200 / R3"
- note added: "Proteccion Cargador\n"
- note added: "Regulador 3.3V"
- note added: "Vprog = 1V"
- moved on the sheet: C10, C6, C7, C8, C9, D3, D4, J1, J11, J12, J13, J15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
